Commit message: Update RL_training: modify URDF, config, demo support, and add pose check scripts

File: RL_training/Isaac_RL/assets/robot_description/urdf/humanoid.urdf (robot description, URDF)
Before this commit: robot humanoid, 22 links, 21 joints
Joints:
- joint left_elbow_pitch_joint: limit lower=-3.14 upper=3.14 effort=20 velocity=50 -> lower=0.000000 upper=2.268928 effort=20 velocity=50
- joint left_wrist_pitch_joint: limit lower=-3.14 upper=3.14 effort=20 velocity=50 -> lower=-2.967060 upper=2.967060 effort=20 velocity=50
- joint right_elbow_pitch_joint: limit lower=-3.14 upper=3.14 effort=20 velocity=50 -> lower=-2.268928 upper=0.000000 effort=20 velocity=50
- joint right_wrist_pitch_joint: limit lower=-3.14 upper=3.14 effort=20 velocity=50 -> lower=-2.967060 upper=2.967060 effort=20 velocity=50
