Commit message: 修改了初始位姿减少奇异点，修改伺服控制为双臂伺服，为符合unity要求，使用实际时钟

File: src/robot_description/urdf/humanoid.urdf (robot description, URDF)
Before this commit: robot humanoid, 22 links, 21 joints
Joints:
- joint right_elbow_pitch_joint: axis -0.333848242516012 0.0592718558412337 0.940761499039 -> 0 0 1; origin xyz=0.0495000377373268 0 0.0624999168897828 rpy=1.5707963267949 0.00263601886731738 1.5707963267949 -> xyz=0.0495000377373268 0 0.0624999168897828 rpy=1.5707963267949 0.456186992961128 1.5707963267949
- joint right_wrist_pitch_joint: axis 0 0 -1 -> 0 0 1

Commit message: fix: sync joint limits from Isaac RL URDF to ROS package (elbow/wrist constraints)

File: src/robot_description/urdf/humanoid.urdf (robot description, URDF)
Before this commit: robot humanoid, 22 links, 21 joints
Joints:
- joint left_elbow_pitch_joint: limit lower=-3.14 upper=3.14 effort=20 velocity=50 -> lower=0.000000 upper=2.268928 effort=20 velocity=50
- joint left_wrist_pitch_joint: limit lower=-3.14 upper=3.14 effort=20 velocity=50 -> lower=-2.967060 upper=2.967060 effort=20 velocity=50
- joint right_elbow_pitch_joint: axis 0 0 1 -> -0.333848242516012 0.0592718558412337 0.940761499039; limit lower=-3.14 upper=3.14 effort=20 velocity=50 -> lower=-2.268928 upper=0.000000 effort=20 velocity=50; origin xyz=0.0495000377373268 0 0.0624999168897828 rpy=1.5707963267949 0.456186992961128 1.5707963267949 -> xyz=0.0495000377373268 0 0.0624999168897828 rpy=1.5707963267949 0.00263601886731738 1.5707963267949
- joint right_wrist_pitch_joint: axis 0 0 1 -> 0 0 -1; limit lower=-3.14 upper=3.14 effort=20 velocity=50 -> lower=-2.967060 upper=2.967060 effort=20 velocity=50

Commit message: modify the axis and the origin of the right elbow pitch joint --htb

File: src/robot_description/urdf/humanoid.urdf (robot description, URDF)
Before this commit: robot humanoid, 22 links, 21 joints
Joints:
- joint right_elbow_pitch_joint: axis -0.333848242516012 0.0592718558412337 0.940761499039 -> 0 0 1; origin xyz=0.0495000377373268 0 0.0624999168897828 rpy=1.5707963267949 0.00263601886731738 1.5707963267949 -> xyz=0.0495000377373268 0 0.0624999168897828 rpy=1.5707963267949 0.456186992961128 1.5707963267949

Commit message: 修改urdf

File: src/robot_description/urdf/humanoid.urdf (robot description, URDF)
Before this commit: robot humanoid, 22 links, 21 joints
Links:
- link base_link: mass 25.2827775843096 -> 25.8765862519602
- link head_camera_link: mass 0.398240212565594 -> 0.0342115541748522
- link left_base_pitch_link: mass 0.244817361510199 -> 0.373968361140818
- link left_camera_link: mass 0.0226998454051643 -> 0.00553667243699105
- link left_elbow_pitch_link: mass 0.154099169383945 -> 0.186600373061323
- link left_gripper1_link: mass 0.0354364112817198 -> 0.0375646671073411
- link left_gripper2_link: mass 0.0354366119716677 -> 0.0375648373217044
- link left_shoulder_roll_link: mass 0.219562602025694 -> 0.344985134468612
- link left_shoulder_yaw_link: mass 0.106143599746768 -> 0.120820726215317
- link left_wrist_pitch_link: mass 0.192205491051058 -> 0.205667966182894
- link left_wrist_yaw_link: mass 0.175099344991619 -> 0.196343643347946
- link neck_pitch_link: mass 0.148218827310183 -> 0.0471064788977039
- link neck_yaw_link: mass 0.0765456211575113 -> 0.682493131271879
- link right_base_pitch_link: mass 0.244817289982652 -> 0.373968361125602
- link right_camera_link: mass 0.0226998455840004 -> 0.00553667243699105
- link right_elbow_pitch_link: mass 0.154099206711241 -> 0.186598823200443
- link right_gripper1_link: mass 0.0358339207664623 -> 0.0375646673398165
- link right_gripper2_link: mass 0.0393551869062514 -> 0.0375648370970392
- link right_shoulder_roll_link: mass 0.219562602027133 -> 0.34498513448704
- link right_shoulder_yaw_link: mass 0.106143604615312 -> 0.12082074165216
- link right_wrist_pitch_link: mass 0.192205595442942 -> 0.205668000586515
- link right_wrist_yaw_link: mass 0.175438598998815 -> 0.196343549066047
Joints:
- joint head_camera_joint: axis (none) -> 0 0 0; origin xyz=0.0498354025053677 0.109164807908296 -0.0267999999999801 rpy=-1.5707963267949 0 0 -> xyz=0.03875 0.14517 -0.021163 rpy=0.070416 1.5708 1.6412
- joint left_base_pitch_joint: origin xyz=-0.213995580451608 0.18999825390085 0.822999049601032 rpy=-1.5707963267949 0 1.5707963267949 -> xyz=0 0.214 0.018 rpy=-1.5708 0 0
- joint left_camera_joint: axis (none) -> 0 0 0; origin xyz=0.000000000 0.071999971 -0.156500000 rpy=-3.141592654 0.000000000 1.570796327 -> xyz=0 -0.072 0.1565 rpy=0 0 -1.5708
- joint left_elbow_pitch_joint: limit lower=0.000000 upper=2.268928 effort=20 velocity=50 -> lower=-3.14 upper=3.14 effort=20 velocity=50; origin xyz=-0.0495001093071362 0 0.0655000777356621 rpy=1.5707963267949 -0.456186992961128 -1.5707963267949 -> xyz=-0.0495 0 0.0625 rpy=1.5708 0 -1.5708
- joint left_gripper1_joint: origin xyz=0 0.14099995082628 -0.0425000000000004 rpy=1.5707963267949 0 -3.14159265358979 -> xyz=0 -0.141 0.0425 rpy=-1.5708 0 3.1416
- joint left_gripper2_joint: origin xyz=0 0.14099995082628 -0.0425000000000004 rpy=1.5707963267949 0 -3.14159265358979 -> xyz=0 -0.141 0.0425 rpy=-1.5708 0 3.1416
- joint left_shoulder_roll_joint: origin xyz=0.0512608845048458 0.00200292781174632 0.0700002065331428 rpy=1.5707963267949 0.0572282794585209 1.6098534872918 -> xyz=0.0513 0 0.07 rpy=1.5708 0 1.5708
- joint left_shoulder_yaw_joint: origin xyz=0.161500206792132 0 -0.0675002120298684 rpy=1.5707963267949 0.127054181766171 1.5707963267949 -> xyz=0.1615 0 -0.0675 rpy=1.5708 0 1.5708
- joint left_wrist_pitch_joint: limit lower=-2.967060 upper=2.967060 effort=20 velocity=50 -> lower=-3.14 upper=3.14 effort=20 velocity=50; origin xyz=0 0.126499835914674 -0.0494999999999997 rpy=1.5707963267949 -0.171337297578539 -3.14159265358979 -> xyz=0 0.1265 -0.0495 rpy=-1.5708 0 0
- joint left_wrist_yaw_joint: origin xyz=0 0.0414999999999796 0.140500028913089 rpy=1.5707963267949 -0.0980347229909209 3.14159265358979 -> xyz=0 -0.0415 0.1405 rpy=-1.5708 0 0
- joint neck_pitch_joint: origin xyz=0 0.189998253900838 0.835499049600994 rpy=1.5707963267949 0 1.5707963267949 -> xyz=0 0 0.0275 rpy=1.5708 0 0
- joint neck_yaw_joint: axis 0 0 1 -> 1 0 0; origin xyz=0.000164597494633156 0.135935192091684 0.0268002104136432 rpy=0 0 0 -> xyz=-0.0001646 0.10793 -0.0331 rpy=0 -1.5708 0
- joint right_base_pitch_joint: axis 0 0 -1 -> 0 0 1; origin xyz=0.21400441954841 0.189998253900819 0.822999049601032 rpy=1.5707963267949 0 1.5707963267949 -> xyz=0 -0.214 0.018 rpy=1.5708 0 0
- joint right_camera_joint: axis (none) -> 0 0 0; origin xyz=0.000000000 0.072000210 -0.156500000 rpy=1.570796327 0.000000000 1.570796327 -> xyz=0 0.072 -0.1565 rpy=1.5708 0 1.5708
- joint right_elbow_pitch_joint: axis -0.333848242516012 0.0592718558412337 0.940761499039 -> 0 0 -1; limit lower=-2.268928 upper=0.000000 effort=20 velocity=50 -> lower=-3.14 upper=3.14 effort=20 velocity=50; origin xyz=0.0495000377373268 0 0.0624999168897828 rpy=1.5707963267949 0.00263601886731738 1.5707963267949 -> xyz=0.0495 0 0.0625 rpy=1.5708 0 1.5708
- joint right_gripper1_joint: axis 1 0 0 -> -1 0 0; limit lower=0 upper=0.03 effort=20 velocity=50 -> lower=-0.03 upper=0 effort=20 velocity=50; origin xyz=0 0.141000000000003 -0.0424999999999999 rpy=1.5707963267949 0 3.14159265358979 -> xyz=0 0.141 -0.0425 rpy=1.5708 0 3.1416
- joint right_gripper2_joint: axis 1 0 0 -> -1 0 0; limit lower=-0.03 upper=0 effort=20 velocity=50 -> lower=0 upper=0.03 effort=20 velocity=50; origin xyz=0 0.141000000000003 -0.0424999999999999 rpy=1.5707963267949 0 3.14159265358979 -> xyz=0 0.141 -0.0425 rpy=1.5708 0 3.1416
- joint right_shoulder_roll_joint: axis 0 0 -1 -> 0 0 1; origin xyz=0.0512767086241353 0.00154568843845215 0.070000086877735 rpy=1.57079632679489 -0.0124370994640314 1.60093654227117 -> xyz=0.0513 0 0.07 rpy=1.5708 0 1.5708
- joint right_shoulder_yaw_joint: origin xyz=-0.161499730454391 0 -0.0674997882054564 rpy=1.5707963267949 -0.209915812016821 -1.5707963267949 -> xyz=-0.1615 0 -0.0675 rpy=1.5708 0 -1.5708
- joint right_wrist_pitch_joint: limit lower=-2.967060 upper=2.967060 effort=20 velocity=50 -> lower=-3.14 upper=3.14 effort=20 velocity=50; origin xyz=0 0.126500083668823 -0.0495002104136634 rpy=1.5707963267949 0.208003209624867 3.14159265358979 -> xyz=0 0.1265 -0.0495 rpy=1.5708 0 3.1416
- joint right_wrist_yaw_joint: origin xyz=0 0.0414999999999797 0.140500210413661 rpy=1.5707963267949 0.575197538261195 3.14159265358979 -> xyz=0 0.0415 0.1405 rpy=1.5708 0 -3.1416

Commit message: Fix the teleoperation issue

File: src/robot_description/urdf/humanoid.urdf (robot description, URDF)
Before this commit: robot humanoid, 22 links, 21 joints
Links:
- added link left_tcp_link
- added link right_tcp_link
Joints:
- added joint left_tcp_joint: type fixed, parent left_wrist_yaw_link, child left_tcp_link, origin xyz=0 0.14099995082628 -0.0425000000000004 rpy=1.5707963267949 0 -3.14159265358979
- added joint right_tcp_joint: type fixed, parent right_wrist_yaw_link, child right_tcp_link, origin xyz=0 0.141000000000003 -0.0424999999999999 rpy=1.5707963267949 0 3.14159265358979

Commit message: Added nodes for moving the robot to the initial position and controlling moveit_servo using the keyboard

File: src/robot_description/urdf/humanoid.urdf (robot description, URDF)
Before this commit: robot humanoid, 24 links, 23 joints
Joints:
- joint right_elbow_pitch_joint: axis 0 0 -1 -> 0 0 1
- joint right_wrist_yaw_joint: axis 0 0 -1 -> 0 0 1

Commit message: modify the robot servol package

File: src/robot_description/urdf/humanoid.urdf (robot description, URDF)
Before this commit: robot humanoid, 24 links, 23 joints
Joints:
- joint left_gripper1_joint: origin xyz=0 0.14099995082628 -0.0425000000000004 rpy=1.5707963267949 0 -3.14159265358979 -> xyz=0 -0.14099995082628 0.0425000000000004 rpy=-1.5707963267949 0 3.14159265358979
- joint left_tcp_joint: origin xyz=0 0.14099995082628 -0.0425000000000004 rpy=1.5707963267949 0 -3.14159265358979 -> xyz=0 -0.14099995082628 0.0425000000000004 rpy=-1.5707963267949 0 3.14159265358979
- joint right_gripper2_joint: axis -1 0 0 -> 1 0 0
- joint right_wrist_pitch_joint: axis 0 0 -1 -> 0 0 1
